Commit message: full model urdf

File: d_bot_description/urdf/d_bot_main.urdf (robot description, URDF)
Before this commit: robot indoor_del_bot, 10 links, 9 joints
Joints:
- joint drive_wheel_left_joint: origin xyz=-7.34417430403589E-06 0.204110516837841 0.0500007440772356 rpy=0 0 0 -> xyz=-7.34417430403589E-06 0.204110516837841 0.0600007440772356 rpy=0 0 0
- joint drive_wheel_right_joint: origin xyz=7.34417430392487E-06 -0.204110516837841 0.0500007440772355 rpy=0 0 0 -> xyz=7.34417430392487E-06 -0.204110516837841 0.0600007440772355 rpy=0 0 0
