Commit message: added sensors

File: d_bot_description/urdf/d_bot_full.xacro (robot description, xacro)
@@ -1,7 +1,9 @@
 <?xml version="1.0"?>
 <robot xmlns:xacro="http://www.ros.org/wiki/xacro" name="d_bot">
+    <!-- include's -->
     <xacro:include filename="$(find d_bot_description)/urdf/caster_transmission.xacro" />
     <xacro:include filename="$(find d_bot_description)/urdf/caster_holder_transmission.xacro" />
-    <xacro:include filename="$(find d_bot_description)/urdf/gazebo.xacro" />
+    <xacro:include filename="$(find d_bot_description)/urdf/gazebo_physics.xacro" />
+    <xacro:include filename="$(find d_bot_description)/urdf/gazebo_sensors.xacro" />
     <xacro:macro name="default_inertial" params="mass">
         <inertial>
@@ -405,5 +407,5 @@
       link="drive_left_link" />
     <axis
-      xyz="1 0 0" />
+      xyz="-1 0 0" />
   </joint>
   <!-- drive_right_link -->
@@ -448,4 +450,30 @@
       xyz="1 0 0" />
   </joint>
+  <!-- imu_link and joint-->
+  <link name="imu_link">
+    <xacro:default_inertial mass="2"/>
+    <visual name="">
+      <origin xyz="0.0 0.0 0.0" rpy="0.0 0.0 0.0"/>
+      <geometry>
+        <box size="0.05 0.05 0.05"/>
+      </geometry>
+      <material name="">
+        <color rgba="1.0 0.0 0.0 1.0"/>
+        <texture filename=""/>
+      </material>
+    </visual>
+    <collision>
+      <origin xyz="0.0 0.0 0.0" rpy="0.0 0.0 0.0"/>
+      <geometry>
+        <box size="0.1 0.1 0.1"/>
+      </geometry>
+    </collision>
+  </link>
+  <joint name="imu_joint" type="fixed">
+    <axis xyz="0 0 0" />
+    <origin xyz="0 0 0.1" rpy="0 0 0"/>
+    <parent link="base_link"/>
+    <child link="imu_link"/>
+  </joint>
 <!-- front_lidar_link -->
   <link
@@ -522,5 +550,5 @@
     <origin
       xyz="0.29154 0.063516 0.2198"
-      rpy="1.4628 0 1.9502" />
+      rpy="1.4628 1.4628 1.9502" />
     <parent
       link="base_link" />

Commit message: collision modified

File: d_bot_description/urdf/d_bot_full.xacro (robot description, xacro)
@@ -6,4 +6,5 @@
     <xacro:include filename="$(find d_bot_description)/urdf/gazebo_physics.xacro" />
     <xacro:include filename="$(find d_bot_description)/urdf/gazebo_sensors.xacro" />
+    <xacro:include filename="$(find d_bot_description)/urdf/gazebo_color.xacro" />
     <xacro:macro name="default_inertial" params="mass">
         <inertial>
@@ -36,5 +37,5 @@
       <geometry>
         <mesh
-          filename="package://d_bot_description/meshes/base_link.STL" />
+          filename="package://d_bot_description/meshes/collision/base_link.STL" />
       </geometry>
     </collision>
@@ -50,5 +51,5 @@
       <geometry>
         <mesh
-          filename="package://d_bot_description/meshes/fl_caster_holder_link.STL" />
+          filename="package://d_bot_description/meshes/caster_holder_link.STL" />
       </geometry>
       <material
@@ -64,5 +65,5 @@
       <geometry>
         <mesh
-          filename="package://d_bot_description/meshes/fl_caster_holder_link.STL" />
+          filename="package://d_bot_description/meshes/collision/caster_holder_link.STL" />
       </geometry>
     </collision>
@@ -91,5 +92,5 @@
       <geometry>
         <mesh
-          filename="package://d_bot_description/meshes/fl_caster_wheel_link.STL" />
+          filename="package://d_bot_description/meshes/caster_wheel_link.STL" />
       </geometry>
       <material
@@ -105,5 +106,5 @@
       <geometry>
         <mesh
-          filename="package://d_bot_description/meshes/fl_caster_wheel_link.STL" />
+          filename="package://d_bot_description/meshes/collision/caster_wheel_link.STL" />
       </geometry>
     </collision>
@@ -132,5 +133,5 @@
       <geometry>
         <mesh
-          filename="package://d_bot_description/meshes/fr_caster_holder_link.STL" />
+          filename="package://d_bot_description/meshes/caster_holder_link.STL" />
       </geometry>
       <material
@@ -146,5 +147,5 @@
       <geometry>
         <mesh
-          filename="package://d_bot_description/meshes/fr_caster_holder_link.STL" />
+          filename="package://d_bot_description/meshes/collision/caster_holder_link.STL" />
       </geometry>
     </collision>
@@ -173,5 +174,5 @@
       <geometry>
         <mesh
-          filename="package://d_bot_description/meshes/fr_caster_wheel_link.STL" />
+          filename="package://d_bot_description/meshes/caster_wheel_link.STL" />
       </geometry>
       <material
@@ -187,5 +188,5 @@
       <geometry>
         <mesh
-          filename="package://d_bot_description/meshes/fr_caster_wheel_link.STL" />
+          filename="package://d_bot_description/meshes/collision/caster_wheel_link.STL" />
       </geometry>
     </collision>
@@ -214,5 +215,5 @@
       <geometry>
         <mesh
-          filename="package://d_bot_description/meshes/bl_caster_holder_link.STL" />
+          filename="package://d_bot_description/meshes/caster_holder_link.STL" />
       </geometry>
       <material
@@ -228,5 +229,5 @@
       <geometry>
         <mesh
-          filename="package://d_bot_description/meshes/bl_caster_holder_link.STL" />
+          filename="package://d_bot_description/meshes/collision/caster_holder_link.STL" />
       </geometry>
     </collision>
@@ -255,5 +256,5 @@
       <geometry>
         <mesh
-          filename="package://d_bot_description/meshes/bl_caster_wheel_link.STL" />
+          filename="package://d_bot_description/meshes/caster_wheel_link.STL" />
       </geometry>
       <material
@@ -269,5 +270,5 @@
       <geometry>
         <mesh
-          filename="package://d_bot_description/meshes/bl_caster_wheel_link.STL" />
+          filename="package://d_bot_description/meshes/collision/caster_wheel_link.STL" />
       </geometry>
     </collision>
@@ -296,5 +297,5 @@
       <geometry>
         <mesh
-          filename="package://d_bot_description/meshes/br_caster_holder_link.STL" />
+          filename="package://d_bot_description/meshes/caster_holder_link.STL" />
       </geometry>
       <material
@@ -310,5 +311,5 @@
       <geometry>
         <mesh
-          filename="package://d_bot_description/meshes/br_caster_holder_link.STL" />
+          filename="package://d_bot_description/meshes/collision/caster_holder_link.STL" />
       </geometry>
     </collision>
@@ -337,5 +338,5 @@
       <geometry>
         <mesh
-          filename="package://d_bot_description/meshes/br_caster_wheel_link.STL" />
+          filename="package://d_bot_description/meshes/caster_wheel_link.STL" />
       </geometry>
       <material
@@ -351,5 +352,5 @@
       <geometry>
         <mesh
-          filename="package://d_bot_description/meshes/br_caster_wheel_link.STL" />
+          filename="package://d_bot_description/meshes/collision/caster_wheel_link.STL" />
       </geometry>
     </collision>
@@ -392,5 +393,5 @@
       <geometry>
         <mesh
-          filename="package://d_bot_description/meshes/drive_left_link.STL" />
+          filename="package://d_bot_description/meshes/collision/drive_left_link.STL" />
       </geometry>
     </collision>
@@ -433,5 +434,5 @@
       <geometry>
         <mesh
-          filename="package://d_bot_description/meshes/drive_right_link.STL" />
+          filename="package://d_bot_description/meshes/collision/drive_right_link.STL" />
       </geometry>
     </collision>
@@ -482,6 +483,6 @@
     <visual>
       <origin
-        xyz="0 0 0"
-        rpy="0 0 0" />
+        xyz="0 0 -0.03"
+        rpy="1.5708 0 1.5708" />
       <geometry>
         <mesh
@@ -496,9 +497,8 @@
     <collision>
       <origin
-        xyz="0 0 0"
-        rpy="0 0 0" />
-      <geometry>
-        <mesh
-          filename="package://d_bot_description/meshes/front_lidar_link.STL" />
+        xyz="-0.05 0 -0.03"
+        rpy="0 0 1.5708" />
+      <geometry>
+        <cylinder radius="0.03" length="0.015"/>
       </geometry>
     </collision>
@@ -508,6 +508,6 @@
     type="fixed">
     <origin
-      xyz="0.32109 0 0.1123"
-      rpy="1.5708 0 1.5708" />
+      xyz="0.32109 0 0.1423"
+      rpy="0 0 0" />
     <parent
       link="base_link" />
@@ -535,5 +535,5 @@
       </material>
     </visual>
-    <collision>
+    <!-- <collision>
       <origin
         xyz="0 0 0"
@@ -543,5 +543,5 @@
           filename="package://d_bot_description/meshes/left_rs_link.STL" />
       </geometry>
-    </collision>
+    </collision> -->
   </link>
   <joint
@@ -550,5 +550,5 @@
     <origin
       xyz="0.29154 0.063516 0.2198"
-      rpy="1.4628 1.4628 1.9502" />
+      rpy="1.4628 0 1.9502" />
     <parent
       link="base_link" />
@@ -576,5 +576,5 @@
       </material>
     </visual>
-    <collision>
+    <!-- <collision>
       <origin
         xyz="0 0 0"
@@ -584,5 +584,5 @@
           filename="package://d_bot_description/meshes/right_rs_link.STL" />
       </geometry>
-    </collision>
+    </collision> -->
   </link>
   <joint

File: d_bot_description/urdf/gazebo_sensors.xacro (robot description, xacro)
@@ -20,4 +20,40 @@
       </plugin>
       <pose>0 0 0 0 0 0</pose>
+    </sensor>
+  </gazebo>
+  <!-- hokuyo -->
+  <gazebo reference="front_lidar_link">
+    <sensor type="ray" name="head_hokuyo_sensor">
+      <pose>0 0 0 0 0 0</pose>
+      <visualize>false</visualize>
+      <update_rate>40</update_rate>
+      <ray>
+        <scan>
+          <horizontal>
+            <samples>720</samples>
+            <resolution>1</resolution>
+            <min_angle>-1.570796</min_angle>
+            <max_angle>1.570796</max_angle>
+          </horizontal>
+        </scan>
+        <range>
+          <min>0.10</min>
+          <max>30.0</max>
+          <resolution>0.01</resolution>
+        </range>
+        <noise>
+          <type>gaussian</type>
+          <!-- Noise parameters based on published spec for Hokuyo laser
+               achieving "+-30mm" accuracy at range < 10m.  A mean of 0.0m and
+               stddev of 0.01m will put 99.7% of samples within 0.03m of the true
+               reading. -->
+          <mean>0.0</mean>
+          <stddev>0.01</stddev>
+        </noise>
+      </ray>
+      <plugin name="gazebo_ros_head_hokuyo_controller" filename="libgazebo_ros_laser.so">
+        <topicName>/rrbot/laser/scan</topicName>
+        <frameName>front_lidar_link</frameName>
+      </plugin>
     </sensor>
   </gazebo>

Commit message: realsense tuning

File: d_bot_description/urdf/d_bot_full.xacro (robot description, xacro)
@@ -523,6 +523,6 @@
     <visual>
       <origin
-        xyz="0 0 0"
-        rpy="0 0 0" />
+        xyz="-0.007 0 0"
+        rpy="1.5708 0 1.7" />
       <geometry>
         <mesh
@@ -549,10 +549,28 @@
     type="fixed">
     <origin
-      xyz="0.29154 0.063516 0.2198"
-      rpy="1.4628 0 1.9502" />
+      xyz="0.3 0.063516 0.2198"
+      rpy="0 0 0.2" />
     <parent
       link="base_link" />
     <child
       link="left_rs_link" />
+    <axis
+      xyz="0 0 0" />
+  </joint>
+  <!-- for visual -->
+  <link
+    name="left_rs_visual_link">
+    <xacro:default_inertial mass="1"/>
+  </link>
+  <joint
+    name="left_rs_visual_joint"
+    type="fixed">
+    <origin
+      xyz="0.3 0.063516 0.2198"
+      rpy="-1.5708 0 -1.3708" />
+    <parent
+      link="base_link" />
+    <child
+      link="left_rs_visual_link" />
     <axis
       xyz="0 0 0" />
@@ -564,6 +582,6 @@
     <visual>
       <origin
-        xyz="0 0 0"
-        rpy="0 0 0" />
+        xyz="-0.007 0 0"
+        rpy="1.46278949747624 0 1.35" />
       <geometry>
         <mesh
@@ -590,10 +608,28 @@
     type="fixed">
     <origin
-      xyz="0.291429416827163 -0.0630797813490415 0.219229621554835"
-      rpy="1.46278949747624 0 1.11167035446073" />
+      xyz="0.3 -0.0630797813490415 0.219229621554835"
+      rpy="0 0 -0.2" />
     <parent
       link="base_link" />
     <child
       link="right_rs_link" />
+    <axis
+      xyz="0 0 0" />
+  </joint>
+  <!-- for visual -->
+  <link
+    name="right_rs_visual_link">
+    <xacro:default_inertial mass="1"/>
+  </link>
+  <joint
+    name="right_rs_visual_joint"
+    type="fixed">
+    <origin
+      xyz="0.3 -0.0630797813490415 0.219229621554835"
+      rpy="-1.5708 0 -1.7708" />
+    <parent
+      link="base_link" />
+    <child
+      link="right_rs_visual_link" />
     <axis
       xyz="0 0 0" />

File: d_bot_description/urdf/gazebo_sensors.xacro (robot description, xacro)
@@ -87,5 +87,50 @@
         <depthImageCameraInfoTopicName>/camera3/depth/camera_info</depthImageCameraInfoTopicName>
         <pointCloudTopicName>/camera3/depth/points</pointCloudTopicName>
-        <frameName>camera_frame_optical_3</frameName>
+        <frameName>left_rs_visual_link</frameName>
+        <pointCloudCutoff>0.01</pointCloudCutoff>
+        <pointCloudCutoffMax>20.0</pointCloudCutoffMax>
+        <distortionK1>0</distortionK1>
+        <distortionK2>0</distortionK2>
+        <distortionK3>0</distortionK3>
+        <distortionT1>0</distortionT1>
+        <distortionT2>0</distortionT2>
+        <CxPrime>0</CxPrime>
+        <Cx>0</Cx>
+        <Cy>0</Cy>
+        <focalLength>0</focalLength>
+        <hackBaseline>0</hackBaseline>
+      </plugin>
+  </sensor>
+</gazebo>
+<!-- Depth camera Left-->
+<gazebo reference="right_rs_link">
+  <sensor type="depth" name="right_camera">
+      <always_on>true</always_on>
+      <visualize>true</visualize>
+      <update_rate>20.0</update_rate>
+      <camera>
+         <horizontal_fov>2.14</horizontal_fov>
+          <image>
+              <format>B8G8R8</format>
+              <width>1280</width>
+              <height>720</height>
+          </image>
+          <clip>
+              <near>0.02</near>
+              <far>12.0</far>
+          </clip>
+      </camera>
+      <plugin name="kinect_camera_controller" filename="libgazebo_ros_openni_kinect.so">
+        <baseline>0.2</baseline>
+        <alwaysOn>true</alwaysOn>
+        <!-- Keep this zero, update_rate in the parent <sensor> tag
+          will control the frame rate. -->
+        <cameraName>camera2</cameraName>
+        <imageTopicName>/camera2/color/image_raw</imageTopicName>
+        <cameraInfoTopicName>/camera2/color/camera_info</cameraInfoTopicName>
+        <depthImageTopicName>/camera2/depth/image_raw</depthImageTopicName>
+        <depthImageCameraInfoTopicName>/camera2/depth/camera_info</depthImageCameraInfoTopicName>
+        <pointCloudTopicName>/camera2/depth/points</pointCloudTopicName>
+        <frameName>right_rs_visual_link</frameName>
         <pointCloudCutoff>0.01</pointCloudCutoff>
         <pointCloudCutoffMax>20.0</pointCloudCutoffMax>
