Commit message: ros2 simulation changes added

File: d_bot_description/urdf/d_bot_full.urdf.xacro (robot description, xacro)
@@ -3,5 +3,5 @@
     <xacro:include filename="$(find d_bot_description)/urdf/caster_transmission.xacro" />
     <xacro:include filename="$(find d_bot_description)/urdf/caster_holder_transmission.xacro" />
-    <xacro:include filename="$(find d_bot_description)/urdf/gazebo.xacro" />
+    <xacro:include filename="$(find d_bot_description)/urdf/robot.gazebo.xacro" />
     <xacro:macro name="default_inertial" params="mass">
         <inertial>
@@ -10,15 +10,29 @@
         </inertial>
     </xacro:macro>
+  <link name="base_footprint"/>
+  <joint
+    name="base_joint"
+    type="fixed">
+    <origin
+      xyz="0.0 0.0 0.0"
+      rpy="0.0 0 0" />
+    <parent
+      link="base_footprint" />
+    <child
+      link="base_link" />
+    <axis
+      xyz="0 0 0" />
+  </joint>
   <!-- base_link -->
   <link
     name="base_link">
-    <xacro:default_inertial mass="100"/>
-    <visual>
-      <origin
-        xyz="0 0 0"
-        rpy="0 0 0" />
-      <geometry>
-        <mesh
-          filename="package://d_bot_description/meshes/base_link.STL" />
+    <xacro:default_inertial mass="10"/>
+    <visual>
+      <origin
+        xyz="0 0 0"
+        rpy="0 0 0" />
+      <geometry>
+        <mesh
+          filename="file:///$(find d_bot_description)/meshes/base_link.STL" />
       </geometry>
       <material
@@ -34,5 +48,5 @@
       <geometry>
         <mesh
-          filename="package://d_bot_description/meshes/base_link.STL" />
+          filename="file:///$(find d_bot_description)/meshes/base_link.STL" />
       </geometry>
     </collision>
@@ -48,5 +62,5 @@
       <geometry>
         <mesh
-          filename="package://d_bot_description/meshes/fl_caster_holder_link.STL" />
+          filename="file:///$(find d_bot_description)/meshes/fl_caster_holder_link.STL" />
       </geometry>
       <material
@@ -62,5 +76,5 @@
       <geometry>
         <mesh
-          filename="package://d_bot_description/meshes/fl_caster_holder_link.STL" />
+          filename="file:///$(find d_bot_description)/meshes/fl_caster_holder_link.STL" />
       </geometry>
     </collision>
@@ -89,5 +103,5 @@
       <geometry>
         <mesh
-          filename="package://d_bot_description/meshes/fl_caster_wheel_link.STL" />
+          filename="file:///$(find d_bot_description)/meshes/fl_caster_wheel_link.STL" />
       </geometry>
       <material
@@ -103,5 +117,5 @@
       <geometry>
         <mesh
-          filename="package://d_bot_description/meshes/fl_caster_wheel_link.STL" />
+          filename="file:///$(find d_bot_description)/meshes/fl_caster_wheel_link.STL" />
       </geometry>
     </collision>
@@ -130,5 +144,5 @@
       <geometry>
         <mesh
-          filename="package://d_bot_description/meshes/fr_caster_holder_link.STL" />
+          filename="file:///$(find d_bot_description)/meshes/fr_caster_holder_link.STL" />
       </geometry>
       <material
@@ -144,5 +158,5 @@
       <geometry>
         <mesh
-          filename="package://d_bot_description/meshes/fr_caster_holder_link.STL" />
+          filename="file:///$(find d_bot_description)/meshes/fr_caster_holder_link.STL" />
       </geometry>
     </collision>
@@ -171,5 +185,5 @@
       <geometry>
         <mesh
-          filename="package://d_bot_description/meshes/fr_caster_wheel_link.STL" />
+          filename="file:///$(find d_bot_description)/meshes/fr_caster_wheel_link.STL" />
       </geometry>
       <material
@@ -185,5 +199,5 @@
       <geometry>
         <mesh
-          filename="package://d_bot_description/meshes/fr_caster_wheel_link.STL" />
+          filename="file:///$(find d_bot_description)/meshes/fr_caster_wheel_link.STL" />
       </geometry>
     </collision>
@@ -212,5 +226,5 @@
       <geometry>
         <mesh
-          filename="package://d_bot_description/meshes/bl_caster_holder_link.STL" />
+          filename="file:///$(find d_bot_description)/meshes/bl_caster_holder_link.STL" />
       </geometry>
       <material
@@ -226,5 +240,5 @@
       <geometry>
         <mesh
-          filename="package://d_bot_description/meshes/bl_caster_holder_link.STL" />
+          filename="file:///$(find d_bot_description)/meshes/bl_caster_holder_link.STL" />
       </geometry>
     </collision>
@@ -253,5 +267,5 @@
       <geometry>
         <mesh
-          filename="package://d_bot_description/meshes/bl_caster_wheel_link.STL" />
+          filename="file:///$(find d_bot_description)/meshes/bl_caster_wheel_link.STL" />
       </geometry>
       <material
@@ -267,5 +281,5 @@
       <geometry>
         <mesh
-          filename="package://d_bot_description/meshes/bl_caster_wheel_link.STL" />
+          filename="file:///$(find d_bot_description)/meshes/bl_caster_wheel_link.STL" />
       </geometry>
     </collision>
@@ -294,5 +308,5 @@
       <geometry>
         <mesh
-          filename="package://d_bot_description/meshes/br_caster_holder_link.STL" />
+          filename="file:///$(find d_bot_description)/meshes/br_caster_holder_link.STL" />
       </geometry>
       <material
@@ -308,5 +322,5 @@
       <geometry>
         <mesh
-          filename="package://d_bot_description/meshes/br_caster_holder_link.STL" />
+          filename="file:///$(find d_bot_description)/meshes/br_caster_holder_link.STL" />
       </geometry>
     </collision>
@@ -335,5 +349,5 @@
       <geometry>
         <mesh
-          filename="package://d_bot_description/meshes/br_caster_wheel_link.STL" />
+          filename="file:///$(find d_bot_description)/meshes/br_caster_wheel_link.STL" />
       </geometry>
       <material
@@ -349,5 +363,5 @@
       <geometry>
         <mesh
-          filename="package://d_bot_description/meshes/br_caster_wheel_link.STL" />
+          filename="file:///$(find d_bot_description)/meshes/br_caster_wheel_link.STL" />
       </geometry>
     </collision>
@@ -376,5 +390,5 @@
       <geometry>
         <mesh
-          filename="package://d_bot_description/meshes/drive_left_link.STL" />
+          filename="file:///$(find d_bot_description)/meshes/drive_left_link.STL" />
       </geometry>
       <material
@@ -390,5 +404,5 @@
       <geometry>
         <mesh
-          filename="package://d_bot_description/meshes/drive_left_link.STL" />
+          filename="file:///$(find d_bot_description)/meshes/drive_left_link.STL" />
       </geometry>
     </collision>
@@ -405,5 +419,5 @@
       link="drive_left_link" />
     <axis
-      xyz="1 0 0" />
+      xyz="-1 0 0" />
   </joint>
   <!-- drive_right_link -->
@@ -417,5 +431,5 @@
       <geometry>
         <mesh
-          filename="package://d_bot_description/meshes/drive_right_link.STL" />
+          filename="file:///$(find d_bot_description)/meshes/drive_right_link.STL" />
       </geometry>
       <material
@@ -431,5 +445,5 @@
       <geometry>
         <mesh
-          filename="package://d_bot_description/meshes/drive_right_link.STL" />
+          filename="file:///$(find d_bot_description)/meshes/drive_right_link.STL" />
       </geometry>
     </collision>
@@ -449,44 +463,21 @@
   </joint>
 <!-- front_lidar_link -->
-  <link
-    name="front_lidar_link">
-    <xacro:default_inertial mass="2"/>
-    <visual>
-      <origin
-        xyz="0 0 0"
-        rpy="0 0 0" />
-      <geometry>
-        <mesh
-          filename="package://d_bot_description/meshes/front_lidar_link.STL" />
-      </geometry>
-      <material
-        name="">
-        <color
-          rgba="0.752941176470588 0.752941176470588 0.752941176470588 0.4" />
-      </material>
-    </visual>
-    <collision>
-      <origin
-        xyz="0 0 0"
-        rpy="0 0 0" />
-      <geometry>
-        <mesh
-          filename="package://d_bot_description/meshes/front_lidar_link.STL" />
-      </geometry>
-    </collision>
-  </link>
-  <joint
-    name="front_lidar_joint"
-    type="fixed">
-    <origin
-      xyz="0.32109 0 0.1123"
-      rpy="1.5708 0 1.5708" />
-    <parent
-      link="base_link" />
-    <child
-      link="front_lidar_link" />
-    <axis
-      xyz="0 0 0" />
-  </joint>
+<joint name="front_lidar_joint" type="fixed">
+        <parent link="base_link"/>
+        <child link="front_lidar_link"/>
+        <origin xyz="0.28109 0 0.13" rpy="0 0 0"/>
+</joint>
+<link name="front_lidar_link">
+    <visual>
+        <geometry>
+            <cylinder radius="0.04" length="0.04"/>
+        </geometry>
+    </visual>
+    <collision>
+        <geometry>
+            <cylinder radius="0.04" length="0.04"/>
+        </geometry>
+    </collision>
+</link>
   <!-- left_rs_link -->
   <link
@@ -496,8 +487,8 @@
       <origin
         xyz="0 0 0"
-        rpy="0 0 0" />
-      <geometry>
-        <mesh
-          filename="package://d_bot_description/meshes/left_rs_link.STL" />
+        rpy="1.5708 0 1.5708" />
+      <geometry>
+        <mesh
+          filename="file:///$(find d_bot_description)/meshes/left_rs_link.STL" />
       </geometry>
       <material
@@ -510,8 +501,8 @@
       <origin
         xyz="0 0 0"
-        rpy="0 0 0" />
-      <geometry>
-        <mesh
-          filename="package://d_bot_description/meshes/left_rs_link.STL" />
+        rpy="1.5708 0 1.5708" />
+      <geometry>
+        <mesh
+          filename="file:///$(find d_bot_description)/meshes/left_rs_link.STL" />
       </geometry>
     </collision>
@@ -522,5 +513,5 @@
     <origin
       xyz="0.29154 0.063516 0.2198"
-      rpy="1.4628 0 1.9502" />
+      rpy="0 0 0.2181662" />
     <parent
       link="base_link" />
@@ -528,5 +519,5 @@
       link="left_rs_link" />
     <axis
-      xyz="0 0 0" />
+      xyz="0 0 0"/>
   </joint>
   <!-- right_rs_link -->
@@ -537,8 +528,8 @@
       <origin
         xyz="0 0 0"
-        rpy="0 0 0" />
-      <geometry>
-        <mesh
-          filename="package://d_bot_description/meshes/right_rs_link.STL" />
+        rpy="1.5708 0 1.5708" />
+      <geometry>
+        <mesh
+          filename="file:///$(find d_bot_description)/meshes/right_rs_link.STL" />
       </geometry>
       <material
@@ -551,8 +542,8 @@
       <origin
         xyz="0 0 0"
-        rpy="0 0 0" />
-      <geometry>
-        <mesh
-          filename="package://d_bot_description/meshes/right_rs_link.STL" />
+        rpy="1.5708 0 1.5708" />
+      <geometry>
+        <mesh
+          filename="file:///$(find d_bot_description)/meshes/right_rs_link.STL" />
       </geometry>
     </collision>
@@ -563,5 +554,5 @@
     <origin
       xyz="0.291429416827163 -0.0630797813490415 0.219229621554835"
-      rpy="1.46278949747624 0 1.11167035446073" />
+      rpy="0 0 -0.2181662" />
     <parent
       link="base_link" />

File: d_bot_description/urdf/d_bot_main.urdf.xacro (robot description, xacro)
@@ -19,5 +19,5 @@
       <geometry>
         <mesh
-          filename="package://d_bot_description/meshes/base_link.STL" />
+          filename="file:///$(find d_bot_description)/meshes/base_link.STL" />
       </geometry>
       <material
@@ -33,5 +33,5 @@
       <geometry>
         <mesh
-          filename="package://d_bot_description/meshes/base_link.STL" />
+          filename="file:///$(find d_bot_description)/meshes/base_link.STL" />
       </geometry>
     </collision>
@@ -60,5 +60,5 @@
       <geometry>
         <mesh
-          filename="package://d_bot_description/meshes/lidar_link.STL" />
+          filename="file:///$(find d_bot_description)/meshes/lidar_link.STL" />
       </geometry>
       <material
@@ -74,5 +74,5 @@
       <geometry>
         <mesh
-          filename="package://d_bot_description/meshes/lidar_link.STL" />
+          filename="file:///$(find d_bot_description)/meshes/lidar_link.STL" />
       </geometry>
     </collision>
@@ -114,5 +114,5 @@
       <geometry>
         <mesh
-          filename="package://d_bot_description/meshes/rs_left.STL" />
+          filename="file:///$(find d_bot_description)/meshes/rs_left.STL" />
       </geometry>
       <material
@@ -128,5 +128,5 @@
       <geometry>
         <mesh
-          filename="package://d_bot_description/meshes/rs_left.STL" />
+          filename="file:///$(find d_bot_description)/meshes/rs_left.STL" />
       </geometry>
     </collision>
@@ -168,5 +168,5 @@
       <geometry>
         <mesh
-          filename="package://d_bot_description/meshes/rs_right.STL" />
+          filename="file:///$(find d_bot_description)/meshes/rs_right.STL" />
       </geometry>
       <material
@@ -182,5 +182,5 @@
       <geometry>
         <mesh
-          filename="package://d_bot_description/meshes/rs_right.STL" />
+          filename="file:///$(find d_bot_description)/meshes/rs_right.STL" />
       </geometry>
     </collision>
@@ -209,5 +209,5 @@
       <geometry>
         <mesh
-          filename="package://d_bot_description/meshes/caster_fl.STL" />
+          filename="file:///$(find d_bot_description)/meshes/caster_fl.STL" />
       </geometry>
       <material
@@ -223,5 +223,5 @@
       <geometry>
         <mesh
-          filename="package://d_bot_description/meshes/caster_fl.STL" />
+          filename="file:///$(find d_bot_description)/meshes/caster_fl.STL" />
       </geometry>
     </collision>
@@ -250,5 +250,5 @@
       <geometry>
         <mesh
-          filename="package://d_bot_description/meshes/caster_fr.STL" />
+          filename="file:///$(find d_bot_description)/meshes/caster_fr.STL" />
       </geometry>
       <material
@@ -264,5 +264,5 @@
       <geometry>
         <mesh
-          filename="package://d_bot_description/meshes/caster_fr.STL" />
+          filename="file:///$(find d_bot_description)/meshes/caster_fr.STL" />
       </geometry>
     </collision>
@@ -291,5 +291,5 @@
       <geometry>
         <mesh
-          filename="package://d_bot_description/meshes/caster_rr.STL" />
+          filename="file:///$(find d_bot_description)/meshes/caster_rr.STL" />
       </geometry>
       <material
@@ -305,5 +305,5 @@
       <geometry>
         <mesh
-          filename="package://d_bot_description/meshes/caster_rr.STL" />
+          filename="file:///$(find d_bot_description)/meshes/caster_rr.STL" />
       </geometry>
     </collision>
@@ -332,5 +332,5 @@
       <geometry>
         <mesh
-          filename="package://d_bot_description/meshes/caster_rl.STL" />
+          filename="file:///$(find d_bot_description)/meshes/caster_rl.STL" />
       </geometry>
       <material
@@ -346,5 +346,5 @@
       <geometry>
         <mesh
-          filename="package://d_bot_description/meshes/caster_rl.STL" />
+          filename="file:///$(find d_bot_description)/meshes/caster_rl.STL" />
       </geometry>
     </collision>
@@ -373,5 +373,5 @@
       <geometry>
         <mesh
-          filename="package://d_bot_description/meshes/drive_wheel_left.STL" />
+          filename="file:///$(find d_bot_description)/meshes/drive_wheel_left.STL" />
       </geometry>
       <material
@@ -387,5 +387,5 @@
       <geometry>
         <mesh
-          filename="package://d_bot_description/meshes/drive_wheel_left.STL" />
+          filename="file:///$(find d_bot_description)/meshes/drive_wheel_left.STL" />
       </geometry>
     </collision>
@@ -415,5 +415,5 @@
       <geometry>
         <mesh
-          filename="package://d_bot_description/meshes/drive_wheel_right.STL" />
+          filename="file:///$(find d_bot_description)/meshes/drive_wheel_right.STL" />
       </geometry>
       <material
@@ -429,5 +429,5 @@
       <geometry>
         <mesh
-          filename="package://d_bot_description/meshes/drive_wheel_right.STL" />
+          filename="file:///$(find d_bot_description)/meshes/drive_wheel_right.STL" />
       </geometry>
     </collision>
@@ -489,8 +489,8 @@
   </transmission>
   <!-- Gazebo plugin for ROS Control -->
-  <gazebo>
+  <!-- <gazebo>
       <plugin name="gazebo_ros_control" filename="libgazebo_ros_control.so">
           <robotNamespace>/</robotNamespace>
       </plugin>
-  </gazebo>
+  </gazebo> -->
 </robot>
