Commit message: cartographer maping added

File: d_bot_description/urdf/d_bot_full.urdf.xacro (robot description, xacro)
@@ -463,11 +463,12 @@
   </joint>
 <!-- front_lidar_link -->
-<joint name="front_lidar_joint" type="fixed">
+<!-- <joint name="front_lidar_joint" type="fixed">
         <parent link="base_link"/>
         <child link="front_lidar_link"/>
-        <origin xyz="0.28109 0 0.13" rpy="0 0 0"/>
+        <origin xyz="0.325 0 0.13" rpy="0 0 0"/>
 </joint>
 <link name="front_lidar_link">
     <visual>
+        <origin xyz="-0.04 0 0" rpy="0 0 0" />
         <geometry>
             <cylinder radius="0.04" length="0.04"/>
@@ -475,9 +476,63 @@
     </visual>
     <collision>
+        <origin xyz="-0.04 0 0" rpy="0 0 0" />
         <geometry>
             <cylinder radius="0.04" length="0.04"/>
         </geometry>
     </collision>
-</link>
+</link> -->
+<link
+    name="lidar_link">
+    <inertial>
+      <origin
+        xyz="0.279194541394812 -1.49381448597552E-05 0.122298548059415"
+        rpy="0 0 0" />
+      <mass
+        value="0.165382751635992" />
+      <inertia
+        ixx="7.88651836105336E-05"
+        ixy="4.84717640920877E-08"
+        ixz="2.18479443959794E-06"
+        iyy="7.51902914938724E-05"
+        iyz="2.88601572510436E-08"
+        izz="0.000109946753058708" />
+    </inertial>
+    <visual>
+      <origin
+        xyz="-0.28 0.0 -0.13"
+        rpy="0 0 0" />
+      <geometry>
+        <mesh
+          filename="file:///$(find d_bot_description)/meshes/lidar_link.STL" />
+      </geometry>
+      <material
+        name="">
+        <color
+          rgba="0.752941176470588 0.752941176470588 0.752941176470588 0.4" />
+      </material>
+    </visual>
+    <collision>
+      <origin
+        xyz="-0.28 0.0 -0.13"
+        rpy="0 0 0" />
+      <geometry>
+        <mesh
+          filename="file:///$(find d_bot_description)/meshes/lidar_link.STL" />
+      </geometry>
+    </collision>
+  </link>
+  <joint
+    name="lidar_joint"
+    type="fixed">
+    <origin
+        xyz="0.2825 0.0 0.13"
+        rpy="0 0 0" />
+    <parent
+      link="base_link" />
+    <child
+      link="lidar_link" />
+    <axis
+      xyz="0 0 0" />
+  </joint>
   <!-- left_rs_link -->
   <link name="left_camera">

File: d_bot_description/urdf/robot.gazebo.xacro (robot description, xacro)
@@ -39,8 +39,8 @@
     </sensor>
   </gazebo>
-  <gazebo reference="front_lidar_link">
+  <gazebo reference="lidar_link">
     <sensor name="laser" type="ray">
       <pose> 0 0 0 0 0 0 </pose>
-      <visualize>false</visualize>
+      <visualize>true</visualize>
       <update_rate>10</update_rate>
       <ray>
@@ -48,10 +48,10 @@
             <horizontal>
                 <samples>360</samples>
-                <min_angle>-3.14</min_angle>
-                <max_angle>3.14</max_angle>
+                <min_angle>-1.74533</min_angle>
+                <max_angle>1.74533</max_angle>
             </horizontal>
         </scan>
         <range>
-            <min>0.3</min>
+            <min>0.05</min>
             <max>12</max>
         </range>
@@ -59,8 +59,8 @@
       <plugin name="laser_controller" filename="libgazebo_ros_ray_sensor.so">
         <ros>
-            <argument>--ros-args --remap ~/out:=scan</argument>
+            <argument>~/out:=scan</argument>
         </ros>
         <output_type>sensor_msgs/LaserScan</output_type>
-        <frame_name>front_lidar_link</frame_name>
+        <frame_name>lidar_link</frame_name>
       </plugin>
     </sensor>

Commit message: collisions changed

File: d_bot_description/urdf/d_bot_full.urdf.xacro (robot description, xacro)
@@ -44,9 +44,36 @@
     <collision>
       <origin
-        xyz="0 0 0"
-        rpy="0 0 0" />
-      <geometry>
-        <mesh
-          filename="file:///$(find d_bot_description)/meshes/base_link.STL" />
+        xyz="-0.05 0 0.18"
+        rpy="0 0 0" />
+      <geometry>
+        <!-- <mesh filename="file:///$(find d_bot_description)/meshes/base_link.STL" /> -->
+        <box size="0.525 0.46 0.1"/>
+      </geometry>
+    </collision>
+    <collision>
+      <origin
+        xyz="0.03 0 0.4"
+        rpy="0 0 0" />
+      <geometry>
+        <!-- <mesh filename="file:///$(find d_bot_description)/meshes/base_link.STL" /> -->
+        <box size="0.64 0.49 0.01"/>
+      </geometry>
+    </collision>
+    <collision>
+      <origin
+        xyz="0.02 0 0.595"
+        rpy="0 0 0" />
+      <geometry>
+        <!-- <mesh filename="file:///$(find d_bot_description)/meshes/base_link.STL" /> -->
+        <box size="0.64 0.49 0.01"/>
+      </geometry>
+    </collision>
+    <collision>
+      <origin
+        xyz="0.01 0 0.79"
+        rpy="0 0 0" />
+      <geometry>
+        <!-- <mesh filename="file:///$(find d_bot_description)/meshes/base_link.STL" /> -->
+        <box size="0.64 0.49 0.01"/>
       </geometry>
     </collision>
@@ -114,8 +141,8 @@
       <origin
         xyz="0 0 0"
-        rpy="0 0 0" />
-      <geometry>
-        <mesh
-          filename="file:///$(find d_bot_description)/meshes/fl_caster_wheel_link.STL" />
+        rpy="0 1.5714 0" />
+      <geometry>
+        <cylinder length="0.02" radius="0.02525"/>
+        <!-- <mesh filename="file:///$(find d_bot_description)/meshes/fl_caster_wheel_link.STL" /> -->
       </geometry>
     </collision>
@@ -196,8 +223,8 @@
       <origin
         xyz="0 0 0"
-        rpy="0 0 0" />
-      <geometry>
-        <mesh
-          filename="file:///$(find d_bot_description)/meshes/fr_caster_wheel_link.STL" />
+        rpy="0 1.5714 0" />
+      <geometry>
+        <cylinder length="0.02" radius="0.02525"/>
+        <!-- <mesh filename="file:///$(find d_bot_description)/meshes/fr_caster_wheel_link.STL" /> -->
       </geometry>
     </collision>
@@ -278,8 +305,8 @@
       <origin
         xyz="0 0 0"
-        rpy="0 0 0" />
-      <geometry>
-        <mesh
-          filename="file:///$(find d_bot_description)/meshes/bl_caster_wheel_link.STL" />
+        rpy="0 1.5714 0" />
+      <geometry>
+        <cylinder length="0.02" radius="0.02525"/>
+        <!-- <mesh filename="file:///$(find d_bot_description)/meshes/bl_caster_wheel_link.STL" /> -->
       </geometry>
     </collision>
@@ -360,8 +387,8 @@
       <origin
         xyz="0 0 0"
-        rpy="0 0 0" />
-      <geometry>
-        <mesh
-          filename="file:///$(find d_bot_description)/meshes/br_caster_wheel_link.STL" />
+        rpy="0 1.5714 0" />
+      <geometry>
+        <cylinder length="0.02" radius="0.02525"/>
+        <!-- <mesh filename="file:///$(find d_bot_description)/meshes/br_caster_wheel_link.STL" /> -->
       </geometry>
     </collision>
@@ -400,9 +427,9 @@
     <collision>
       <origin
-        xyz="0 0 0"
-        rpy="0 0 0" />
-      <geometry>
-        <mesh
-          filename="file:///$(find d_bot_description)/meshes/drive_left_link.STL" />
+        xyz="0.05 0 0"
+        rpy="0 1.5714 0" />
+      <geometry>
+        <!-- <mesh filename="file:///$(find d_bot_description)/meshes/drive_left_link.STL" /> -->
+        <cylinder length="0.05" radius="0.0825"/>
       </geometry>
     </collision>
@@ -441,9 +468,9 @@
     <collision>
       <origin
-        xyz="0 0 0"
-        rpy="0 0 0" />
-      <geometry>
-        <mesh
-          filename="file:///$(find d_bot_description)/meshes/drive_right_link.STL" />
+        xyz="0.05 0 0"
+        rpy="0 1.5714 0" />
+      <geometry>
+      <cylinder length="0.05" radius="0.0825"/>
+        <!-- <mesh filename="file:///$(find d_bot_description)/meshes/drive_right_link.STL" /> -->
       </geometry>
     </collision>
@@ -649,5 +676,5 @@
       <origin xyz="0.0 0.0 0.0" rpy="0.0 0.0 0.0"/>
       <geometry>
-        <box size="0.1 0.1 0.1"/>
+        <box size="0.05 0.05 0.05"/>
       </geometry>
     </collision>
@@ -655,5 +682,5 @@
   <joint name="imu_joint" type="fixed">
     <axis xyz="0 0 0" />
-    <origin xyz="0 0 0.1" rpy="0 0 0"/>
+    <origin xyz="0 0 0.26" rpy="0 0 0"/>
     <parent link="base_link"/>
     <child link="imu_link"/>
